Commit message: imporved launch and urdf files

File: ros_ws/src/efim/efim.urdf (robot description, URDF)
Before this commit: robot efim, 7 links, 6 joints
Links:
- link wheel_front_left: geometry collision cylinder length=0.0508 radius=0.0762; visual cylinder length=0.0508 radius=0.0762
- link wheel_front_right: geometry collision cylinder length=0.0508 radius=0.0762; visual cylinder length=0.0508 radius=0.0762
- link wheel_rear_left: geometry collision cylinder length=0.0508 radius=0.0762; visual cylinder length=0.0508 radius=0.0762
- link wheel_rear_right: geometry collision cylinder length=0.0508 radius=0.0762; visual cylinder length=0.0508 radius=0.0762
Joints:
- removed joint axiz_front_left
- removed joint axiz_front_right
- removed joint axiz_rear_left
- removed joint axiz_rear_right
- added joint axis_front_left: type continuous, parent base_lower_link, child wheel_front_left, origin xyz=0.165862 0.18034 0 rpy=-1.5708 0 0, axis 0 0 1
- added joint axis_front_right: type continuous, parent base_lower_link, child wheel_front_right, origin xyz=0.165862 -0.18034 0 rpy=-1.5708 0 0, axis 0 0 1
- added joint axis_rear_left: type continuous, parent base_lower_link, child wheel_rear_left, origin xyz=-0.165862 0.18034 0 rpy=-1.5708 0 0, axis 0 0 1
- added joint axis_rear_right: type continuous, parent base_lower_link, child wheel_rear_right, origin xyz=-0.165862 -0.18034 0 rpy=-1.5708 0 0, axis 0 0 1

Commit message: odom transforms now working

File: ros_ws/src/efim/efim.urdf (robot description, URDF)
Before this commit: robot efim, 7 links, 6 joints
Links:
- removed link base_lower_link
- added link body_link, mass 12.0; collision cylinder length=1.04775 radius=0.2032; visual cylinder length=1.04775 radius=0.2032
- added link laser_link, mass 0.25; collision box size=0.2794 0.0762 0.0762; visual box size=0.0762 0.2794 0.0762
- link base_link: mass 12.0 -> 16.0; geometry collision box size=0.41148 0.30988 0.05588; visual box size=0.41148 0.30988 0.05588
Joints:
- added joint laser_joint: type fixed, parent body_link, child laser_link, origin xyz=0.2032 0 0 rpy=0 0 0, axis 0 0 1
- joint axis_front_left: parent base_lower_link -> base_link
- joint axis_front_right: parent base_lower_link -> base_link
- joint axis_rear_left: parent base_lower_link -> base_link
- joint axis_rear_right: parent base_lower_link -> base_link
- joint center_joint: child base_lower_link -> body_link; origin xyz=0 0 -0.551815 rpy=0 0 0 -> xyz=0 0 0.551815 rpy=0 0 0; type continuous -> fixed
- joint hitch_joint: parent base_lower_link -> base_link

Commit message: Updated launch files

File: ros_ws/src/efim/efim.urdf (robot description, URDF)
Before this commit: robot efim, 8 links, 7 joints
Links:
- link laser_link: geometry collision box size=0.0762 0.2794 0.0762; visual box size=0.0762 0.2794 0.0762
Joints:
- joint laser_joint: origin xyz=0.2032 0 0 rpy=0 0 0 -> xyz=0.2032 0 -0.3 rpy=0 0 0

Commit message: Updated configs

File: ros_ws/src/efim/efim.urdf (robot description, URDF)
Before this commit: robot efim, 8 links, 7 joints
Links:
- link base_link: mass 16.0 -> 20.0
- link body_link: mass 12.0 -> 10.0
Joints:
- joint laser_joint: origin xyz=0.2032 0 -0.3 rpy=0 0 0 -> xyz=0.2 0 -0.3 rpy=0 0 0
