Commit message: improved navigation

File: ros_ws/src/efim/efim.urdf.xacro (robot description, xacro)
@@ -1,4 +1,8 @@
 <?xml version="1.0"?>
-<robot name="efim">
+<robot name="efim"
+       xmlns:sensor="http://playerstage.sourceforge.net/gazebo/xmlschema/#sensor"
+       xmlns:controller="http://playerstage.sourceforge.net/gazebo/xmlschema/#controller"
+       xmlns:interface="http://playerstage.sourceforge.net/gazebo/xmlschema/#interface"
+       xmlns:xacro="http://ros.org/wiki/xacro">
   <link name="base_link">
     <visual>
@@ -70,6 +74,45 @@
     </inertial>
   </link>
-<gazebo reference="laser_link">
-    <sensor type="depth" name="openni_camera_camera">
+<!--<xacro:macro name="sim_kinect">
+   <gazebo reference="laser_link">
+      <sensor type="depth" name="camera">
+        <always_on>true</always_on>
+        <update_rate>20.0</update_rate>
+        <camera>
+          <horizontal_fov>${60.0*3.14/180.0}</horizontal_fov>
+          <image>
+            <format>R8G8B8</format>
+            <width>640</width>
+            <height>480</height>
+          </image>
+          <clip>
+            <near>0.05</near>
+            <far>8.0</far>
+          </clip>
+        </camera>
+        <plugin name="kinect_camera_controller" filename="libgazebo_ros_openni_kinect.so">
+          <cameraName>camera</cameraName>
+          <alwaysOn>true</alwaysOn>
+          <updateRate>10</updateRate>
+          <imageTopicName>rgb/image_raw</imageTopicName>
+          <depthImageTopicName>depth/image_raw</depthImageTopicName>
+          <pointCloudTopicName>depth/points</pointCloudTopicName>
+          <cameraInfoTopicName>rgb/camera_info</cameraInfoTopicName>
+          <depthImageCameraInfoTopicName>depth/camera_info</depthImageCameraInfoTopicName>
+          <frameName>camera_depth_optical_frame</frameName>
+          <baseline>0.1</baseline>
+          <distortion_k1>0.0</distortion_k1>
+          <distortion_k2>0.0</distortion_k2>
+          <distortion_k3>0.0</distortion_k3>
+          <distortion_t1>0.0</distortion_t1>
+          <distortion_t2>0.0</distortion_t2>
+          <pointCloudCutoff>0.4</pointCloudCutoff>
+        </plugin>
+      </sensor>
+    </gazebo>
+</xacro:macro>
+<sim_kinect/>-->
+<!--<gazebo reference="laser_link">
+    <sensor type="depth" name="camera">
         <always_on>1</always_on>
         <visualize>true</visualize>
@@ -84,9 +127,10 @@
             </depth_camera>
             <clip>
-                <near>0.1</near>
-                <far>100</far>
+                <near>0.05</near>
+                <far>8.0</far>
             </clip>
         </camera>
         <plugin name="camera_controller" filename="libgazebo_ros_openni_kinect.so">
+            <cameraName>camera</cameraName>
             <alwaysOn>true</alwaysOn>
                 <updateRate>10.0</updateRate>
@@ -111,6 +155,6 @@
             </plugin>
     </sensor>
-</gazebo>
- <!-- <gazebo reference="laser_link">
+</gazebo>-->
+ <gazebo reference="laser_link">
     <material>Gazebo/Blue</material>
     <sensor type="gpu_ray" name="hokuyo">
@@ -138,5 +182,5 @@
       </plugin>
     </sensor>
-  </gazebo> -->
+  </gazebo>
   <joint name="laser_joint" type="fixed">
     <axis xyz="0 0 1"/>

Commit message: changed laser_link to camera_link

File: ros_ws/src/efim/efim.urdf.xacro (robot description, xacro)
@@ -54,5 +54,5 @@
     <origin rpy="0 0 0" xyz="0 0 0.551815"/>
   </joint>
-  <link name="laser_link">
+  <link name="camera_link">
     <visual>
       <geometry>
@@ -75,5 +75,5 @@
   </link>
 <!--<xacro:macro name="sim_kinect">
-   <gazebo reference="laser_link">
+   <gazebo reference="camera_link">
       <sensor type="depth" name="camera">
         <always_on>true</always_on>
@@ -100,5 +100,5 @@
           <cameraInfoTopicName>rgb/camera_info</cameraInfoTopicName>
           <depthImageCameraInfoTopicName>depth/camera_info</depthImageCameraInfoTopicName>
-          <frameName>laser_link</frameName>
+          <frameName>camera_link</frameName>
           <baseline>0.1</baseline>
           <distortion_k1>0.0</distortion_k1>
@@ -113,5 +113,5 @@
 </xacro:macro>
 <sim_kinect/>-->
-<!--<gazebo reference="laser_link">
+<gazebo reference="camera_link">
     <sensor type="depth" name="camera">
         <always_on>1</always_on>
@@ -136,7 +136,7 @@
                 <updateRate>10.0</updateRate>
                 <cameraName>camera</cameraName>
-                <frameName>laser_link</frameName>
+                <frameName>camera_link</frameName>
             <imageTopicName>rgb/image_raw</imageTopicName>
-            <depthImageTopicName>depth/image_raw</depthImageTopicName>
+            <depthImageTopicName>depth_registered/image_raw</depthImageTopicName>
             <pointCloudTopicName>depth/points</pointCloudTopicName>
             <cameraInfoTopicName>rgb/camera_info</cameraInfoTopicName>
@@ -155,6 +155,6 @@
             </plugin>
     </sensor>
-</gazebo>-->
- <gazebo reference="laser_link">
+</gazebo>
+<!-- <gazebo reference="camera_link">
     <material>Gazebo/Blue</material>
     <sensor type="gpu_ray" name="hokuyo">
@@ -179,12 +179,12 @@
       <plugin name="gpu_laser" filename="libgazebo_ros_gpu_laser.so">
         <topicName>/scan</topicName>
-        <frameName>laser_link</frameName>
+        <frameName>camera_link</frameName>
       </plugin>
     </sensor>
-  </gazebo>
+  </gazebo> -->
   <joint name="laser_joint" type="fixed">
     <axis xyz="0 0 1"/>
     <parent link="body_link"/>
-    <child link="laser_link"/>
+    <child link="camera_link"/>
     <origin rpy="0 0 0" xyz="0.2 0 -0.3"/>
   </joint>

Commit message: updates

File: ros_ws/src/efim/efim.urdf.xacro (robot description, xacro)
@@ -183,9 +183,35 @@
     </sensor>
   </gazebo> -->
-  <joint name="laser_joint" type="fixed">
+  <joint name="camera_joint" type="fixed">
     <axis xyz="0 0 1"/>
     <parent link="body_link"/>
     <child link="camera_link"/>
     <origin rpy="0 0 0" xyz="0.2 0 -0.3"/>
+  </joint>
+  <link name="laser">
+    <visual>
+      <geometry>
+        <box size="0.0762 0.2794 0.0762"/>
+      </geometry>
+      <material name="blue">
+	<color rgba="0.1 0.1 1 1"/>
+      </material>
+    </visual>
+    <collision>
+      <geometry>
+        <box size="0.0762 0.2794 0.0762"/>
+      </geometry>
+    </collision>
+   <inertial>
+      <mass value="0.25"/>
+      <inertia ixx="1.0" iyy="1.0" izz="1.0"
+               ixy="0" ixz="0" iyz="0"/>
+    </inertial>
+  </link>
+  <joint name="laser_joint" type="fixed">
+    <axis xyz="0 0 1"/>
+    <parent link="body_link"/>
+    <child link="laser"/>
+    <origin rpy="0 0 0" xyz="0.2 0 0.5"/>
   </joint>
   <link name="hitch_front_link">

Commit message: Laser odom working

File: ros_ws/src/efim/efim.urdf.xacro (robot description, xacro)
@@ -48,5 +48,5 @@
     </inertial>
   </link>
-  <joint name="center_joint" type="fixed">
+  <joint name="center_joint" type="continuous">
     <axis xyz="0 0 1"/>
     <parent link="base_link"/>
@@ -198,9 +198,9 @@
       </material>
     </visual>
-    <collision>
+    <!--<collision>
       <geometry>
         <box size="0.0762 0.2794 0.0762"/>
       </geometry>
-    </collision>
+    </collision>-->
    <inertial>
       <mass value="0.25"/>
@@ -209,7 +209,7 @@
     </inertial>
   </link>
-  <joint name="laser_joint" type="fixed">
-    <axis xyz="0 0 1"/>
-    <parent link="body_link"/>
+  <joint name="laser_joint" type="continuous">
+    <axis xyz="0 0 1"/>
+    <parent link="base_link"/>
     <child link="laser"/>
     <origin rpy="0 0 0" xyz="0.2 0 0.5"/>

Commit message: RTABMap working

File: ros_ws/src/efim/efim.urdf.xacro (robot description, xacro)
@@ -74,45 +74,6 @@
     </inertial>
   </link>
-<!--<xacro:macro name="sim_kinect">
-   <gazebo reference="camera_link">
-      <sensor type="depth" name="camera">
-        <always_on>true</always_on>
-        <update_rate>20.0</update_rate>
-        <camera>
-          <horizontal_fov>${60.0*3.14/180.0}</horizontal_fov>
-          <image>
-            <format>R8G8B8</format>
-            <width>640</width>
-            <height>480</height>
-          </image>
-          <clip>
-            <near>0.05</near>
-            <far>8.0</far>
-          </clip>
-        </camera>
-        <plugin name="kinect_camera_controller" filename="libgazebo_ros_openni_kinect.so">
-          <cameraName>camera</cameraName>
-          <alwaysOn>true</alwaysOn>
-          <updateRate>10</updateRate>
-          <imageTopicName>rgb/image_raw</imageTopicName>
-          <depthImageTopicName>depth/image_raw</depthImageTopicName>
-          <pointCloudTopicName>depth/points</pointCloudTopicName>
-          <cameraInfoTopicName>rgb/camera_info</cameraInfoTopicName>
-          <depthImageCameraInfoTopicName>depth/camera_info</depthImageCameraInfoTopicName>
-          <frameName>camera_link</frameName>
-          <baseline>0.1</baseline>
-          <distortion_k1>0.0</distortion_k1>
-          <distortion_k2>0.0</distortion_k2>
-          <distortion_k3>0.0</distortion_k3>
-          <distortion_t1>0.0</distortion_t1>
-          <distortion_t2>0.0</distortion_t2>
-          <pointCloudCutoff>0.4</pointCloudCutoff>
-        </plugin>
-      </sensor>
-    </gazebo>
-</xacro:macro>
-<sim_kinect/>-->
 <gazebo reference="camera_link">
-    <sensor type="depth" name="camera">
+    <sensor type="depth" name="camera_link">
         <always_on>1</always_on>
         <visualize>true</visualize>
@@ -136,5 +97,5 @@
                 <updateRate>10.0</updateRate>
                 <cameraName>camera</cameraName>
-                <frameName>camera_link</frameName>
+                <frameName>camera</frameName>
             <imageTopicName>rgb/image_raw</imageTopicName>
             <depthImageTopicName>depth_registered/image_raw</depthImageTopicName>
@@ -156,32 +117,5 @@
     </sensor>
 </gazebo>
-<!-- <gazebo reference="camera_link">
-    <material>Gazebo/Blue</material>
-    <sensor type="gpu_ray" name="hokuyo">
-      <pose>0 0 0 0 0 0</pose>
-      <visualize>true</visualize>
-      <update_rate>40</update_rate>
-      <ray>
-        <scan>
-          <horizontal>
-            <samples>720</samples>
-            <resolution>1</resolution>
-            <min_angle>-1.570796</min_angle>
-            <max_angle>1.570796</max_angle>
-          </horizontal>
-        </scan>
-        <range>
-          <min>0.10</min>
-          <max>30.0</max>
-          <resolution>0.01</resolution>
-        </range>
-      </ray>
-      <plugin name="gpu_laser" filename="libgazebo_ros_gpu_laser.so">
-        <topicName>/scan</topicName>
-        <frameName>camera_link</frameName>
-      </plugin>
-    </sensor>
-  </gazebo> -->
-  <joint name="camera_joint" type="fixed">
+  <joint name="camera_joint" type="continuous">
     <axis xyz="0 0 1"/>
     <parent link="body_link"/>

Commit message: Moved lasers

File: ros_ws/src/efim/efim.urdf.xacro (robot description, xacro)
@@ -145,7 +145,7 @@
   <joint name="laser_joint" type="continuous">
     <axis xyz="0 0 1"/>
-    <parent link="base_link"/>
+    <parent link="body_link"/>
     <child link="laser"/>
-    <origin rpy="0 0 0" xyz="0.2 0 0.5"/>
+    <origin rpy="0 0 0" xyz="0.0 0 0.55"/>
   </joint>
   <link name="hitch_front_link">
