Commit message: updates

File: ros/urdf/efim.urdf.xacro (robot description, xacro)
@@ -95,8 +95,7 @@
             <cameraName>camera</cameraName>
             <alwaysOn>true</alwaysOn>
-                <updateRate>10.0</updateRate>
-                <cameraName>camera</cameraName>
-                <frameName>camera</frameName>
-            <imageTopicName>rgb/image_raw</imageTopicName>
+            <updateRate>10.0</updateRate>
+            <frameName>camera_link</frameName>
+            <imageTopicName>rgb/image_rect_color</imageTopicName>
             <depthImageTopicName>depth_registered/image_raw</depthImageTopicName>
             <pointCloudTopicName>depth/points</pointCloudTopicName>
@@ -104,15 +103,15 @@
             <depthImageCameraInfoTopicName>depth/camera_info</depthImageCameraInfoTopicName>
             <pointCloudCutoff>0.4</pointCloudCutoff>
-                <hackBaseline>0.07</hackBaseline>
-                <distortionK1>0.0</distortionK1>
-                <distortionK2>0.0</distortionK2>
-                <distortionK3>0.0</distortionK3>
-                <distortionT1>0.0</distortionT1>
-                <distortionT2>0.0</distortionT2>
+            <hackBaseline>0.07</hackBaseline>
+            <distortionK1>0.0</distortionK1>
+            <distortionK2>0.0</distortionK2>
+            <distortionK3>0.0</distortionK3>
+            <distortionT1>0.0</distortionT1>
+            <distortionT2>0.0</distortionT2>
             <CxPrime>0.0</CxPrime>
             <Cx>0.0</Cx>
             <Cy>0.0</Cy>
             <focalLength>0.0</focalLength>
-            </plugin>
+        </plugin>
     </sensor>
 </gazebo>
@@ -279,5 +278,5 @@
   <plugin name="skid_steer_drive_controller" filename="libgazebo_ros_skid_steer_drive.so">
     <updateRate>100.0</updateRate>
-    <robotNamespace>/</robotNamespace>
+    <robotNamespace></robotNamespace>
     <leftFrontJoint>axis_front_left</leftFrontJoint>
     <rightFrontJoint>axis_front_right</rightFrontJoint>
@@ -290,8 +289,38 @@
     <commandTopic>cmd_vel</commandTopic>
     <broadcastTF>1</broadcastTF>
+    <odometryFrame>/odom_frame_gazebo</odometryFrame>
+    <odometryTopic>/odom_gazebo</odometryTopic>
   </plugin>
   <plugin name="joint_state_publisher" filename="libgazebo_ros_joint_state_publisher.so">
     <jointName>axis_front_left, axis_front_right, axis_rear_left, axis_rear_right</jointName>
+    <updateRate>100</updateRate>
   </plugin>
 </gazebo>
+<gazebo reference="laser">
+    <material>Gazebo/Blue</material>
+    <sensor type="ray" name="head_hokuyo_sensor">
+      <pose>0 0 0 0 0 0</pose>
+      <visualize>true</visualize>
+      <update_rate>40</update_rate>
+      <ray>
+        <scan>
+          <horizontal>
+            <samples>720</samples>
+            <resolution>1</resolution>
+            <min_angle>-1.570795</min_angle>
+            <max_angle>1.570795</max_angle>
+          </horizontal>
+        </scan>
+        <range>
+          <min>0.10</min>
+          <max>30.0</max>
+          <resolution>0.01</resolution>
+        </range>
+      </ray>
+      <plugin name="gazebo_ros_head_hokuyo_controller" filename="libgazebo_ros_laser.so">
+        <topicName>/scan</topicName>
+        <frameName>laser</frameName>
+      </plugin>
+    </sensor>
+  </gazebo>
 </robot>

Commit message: update

File: ros/urdf/efim.urdf.xacro (robot description, xacro)
@@ -37,9 +37,9 @@
       </material>
     </visual>
-    <collision>
+    <!--<collision>
       <geometry>
         <cylinder length="1.04775" radius="0.2032"/>
       </geometry>
-    </collision>
+    </collision>-->
     <inertial>
       <mass value="10.0"/>
@@ -48,5 +48,5 @@
     </inertial>
   </link>
-  <joint name="center_joint" type="continuous">
+  <joint name="center_joint" type="fixed">
     <axis xyz="0 0 1"/>
     <parent link="base_link"/>
@@ -63,9 +63,9 @@
       </material>
     </visual>
-    <collision>
+    <!--<collision>
       <geometry>
         <box size="0.0762 0.2794 0.0762"/>
       </geometry>
-    </collision>
+    </collision>-->
    <inertial>
       <mass value="0.25"/>
@@ -74,5 +74,214 @@
     </inertial>
   </link>
-<gazebo reference="camera_link">
+  <joint name="camera_joint" type="continuous">
+    <axis xyz="0 0 0"/>
+    <parent link="body_link"/>
+    <child link="camera_link"/>
+    <origin rpy="0 0 0" xyz="0.4 0 -0.3"/>
+  </joint>
+  <link name="laser">
+    <visual>
+      <geometry>
+        <box size="0.0762 0.2794 0.0762"/>
+      </geometry>
+      <material name="blue">
+	<color rgba="0.1 0.1 1 1"/>
+      </material>
+    </visual>
+    <!--<collision>
+      <geometry>
+        <box size="0.0762 0.2794 0.0762"/>
+      </geometry>
+    </collision>-->
+   <inertial>
+      <mass value="0.25"/>
+      <inertia ixx="1.0" iyy="1.0" izz="1.0"
+               ixy="0" ixz="0" iyz="0"/>
+    </inertial>
+  </link>
+  <joint name="laser_joint" type="fixed">
+    <axis xyz="0 0 1"/>
+    <parent link="body_link"/>
+    <child link="laser"/>
+    <origin rpy="0 0 0" xyz="0.0 0 0.55"/>
+  </joint>
+  <link name="hitch_front_link">
+    <visual>
+      <geometry>
+        <cylinder length="0.1524" radius="0.01"/>
+      </geometry>
+      <material name="silver">
+	<color rgba="0.75 0.75 0.75 1"/>
+      </material>
+    </visual>
+    <collision>
+      <geometry>
+        <cylinder length="0.1524" radius="0.01"/>
+      </geometry>
+    </collision>
+    <inertial>
+      <mass value="0.1"/>
+      <inertia ixx="1.0" iyy="1.0" izz="1.0"
+               ixy="0" ixz="0" iyz="0"/>
+    </inertial>
+  </link>
+  <joint name="hitch_joint" type="fixed">
+    <axis xyz="0 0 1"/>
+    <parent link="base_link"/>
+    <child link="hitch_front_link"/>
+    <origin rpy="0 0 0" xyz="0.18 0 0.0762"/>
+  </joint>
+  <link name="wheel_front_left">
+    <visual>
+      <geometry>
+        <cylinder length="0.0508" radius="0.0762"/>
+      </geometry>
+      <material name="black">
+        <color rgba="0 0 0 1"/>
+      </material>
+    </visual>
+    <collision>
+      <geometry>
+        <cylinder length="0.0508" radius="0.0762"/>
+      </geometry>
+    </collision>
+    <inertial>
+      <mass value="0.1"/>
+      <inertia ixx="1.0" iyy="1.0" izz="1.0"
+               ixy="0" ixz="0" iyz="0"/>
+    </inertial>
+  </link>
+  <joint name="axis_front_left" type="continuous">
+    <axis xyz="0 0 1"/>
+    <parent link="base_link"/>
+    <child link="wheel_front_left"/>
+    <origin rpy="-1.5708 0 0" xyz="0.165862 0.18034 0"/>
+  </joint>
+ <link name="wheel_front_right">
+    <visual>
+      <geometry>
+        <cylinder length="0.0508" radius="0.0762"/>
+      </geometry>
+      <material name="black"/>
+    </visual>
+    <collision>
+      <geometry>
+        <cylinder length="0.0508" radius="0.0762"/>
+      </geometry>
+    </collision>
+    <inertial>
+      <mass value="0.1"/>
+      <inertia ixx="1.0" iyy="1.0" izz="1.0"
+               ixy="0" ixz="0" iyz="0"/>
+    </inertial>
+  </link>
+  <joint name="axis_front_right" type="continuous">
+    <axis xyz="0 0 1"/>
+    <parent link="base_link"/>
+    <child link="wheel_front_right"/>
+    <origin rpy="-1.5708 0 0" xyz="0.165862 -0.18034 0"/>
+  </joint>
+  <link name="wheel_rear_right">
+    <visual>
+      <geometry>
+        <cylinder length="0.0508" radius="0.0762"/>
+      </geometry>
+      <material name="black"/>
+    </visual>
+    <collision>
+      <geometry>
+        <cylinder length="0.0508" radius="0.0762"/>
+      </geometry>
+    </collision>
+    <inertial>
+      <mass value="0.1"/>
+      <inertia ixx="1.0" iyy="1.0" izz="1.0"
+               ixy="0" ixz="0" iyz="0"/>
+    </inertial>
+  </link>
+  <joint name="axis_rear_right" type="continuous">
+    <axis xyz="0 0 1"/>
+    <parent link="base_link"/>
+    <child link="wheel_rear_right"/>
+    <origin rpy="-1.5708 0 0" xyz="-0.165862 -0.18034 0"/>
+  </joint>
+  <link name="wheel_rear_left">
+    <visual>
+      <geometry>
+        <cylinder length="0.0508" radius="0.0762"/>
+      </geometry>
+      <material name="black"/>
+    </visual>
+    <collision>
+      <geometry>
+        <cylinder length="0.0508" radius="0.0762"/>
+      </geometry>
+    </collision>
+    <inertial>
+      <mass value="0.1"/>
+      <inertia ixx="1.0" iyy="1.0" izz="1.0"
+               ixy="0" ixz="0" iyz="0"/>
+    </inertial>
+    <gazebo reference="wheel_rear_left">
+      <material>Gazebo/Black</material>
+    </gazebo>
+  </link>
+  <joint name="axis_rear_left" type="continuous">
+    <axis xyz="0 0 1"/>
+    <parent link="base_link"/>
+    <child link="wheel_rear_left"/>
+    <origin rpy="-1.5708 0 0" xyz="-0.165862 0.18034 0"/>
+  </joint>
+<gazebo>
+  <plugin name="skid_steer_drive_controller" filename="libgazebo_ros_skid_steer_drive.so">
+    <updateRate>100.0</updateRate>
+    <robotNamespace></robotNamespace>
+    <leftFrontJoint>axis_front_left</leftFrontJoint>
+    <rightFrontJoint>axis_front_right</rightFrontJoint>
+    <leftRearJoint>axis_rear_left</leftRearJoint>
+    <rightRearJoint>axis_rear_right</rightRearJoint>
+    <wheelSeparation>0.254</wheelSeparation>
+    <wheelDiameter>0.1524</wheelDiameter>
+    <robotBaseFrame>base_link</robotBaseFrame>
+    <torque>10</torque>
+    <commandTopic>cmd_vel</commandTopic>
+    <broadcastTF>0</broadcastTF>
+    <odometryFrame>/odom_frame_gazebo</odometryFrame>
+    <odometryTopic>/odom_gazebo</odometryTopic>
+  </plugin>
+  <plugin name="joint_state_publisher" filename="libgazebo_ros_joint_state_publisher.so">
+    <jointName>axis_front_left, axis_front_right, axis_rear_left, axis_rear_right</jointName>
+    <updateRate>100</updateRate>
+  </plugin>
+</gazebo>
+<gazebo reference="laser">
+    <material>Gazebo/Blue</material>
+    <sensor type="gpu_ray" name="head_hokuyo_sensor">
+      <pose>0 0 0 0 0 0</pose>
+      <visualize>true</visualize>
+      <update_rate>40</update_rate>
+      <ray>
+        <scan>
+          <horizontal>
+            <samples>720</samples>
+            <resolution>1</resolution>
+            <min_angle>-1.570795</min_angle>
+            <max_angle>1.570795</max_angle>
+          </horizontal>
+        </scan>
+        <range>
+          <min>0.10</min>
+          <max>30.0</max>
+          <resolution>0.01</resolution>
+        </range>
+      </ray>
+      <plugin name="gazebo_ros_head_hokuyo_controller" filename="libgazebo_ros_gpu_laser.so">
+        <topicName>/scan</topicName>
+        <frameName>laser</frameName>
+      </plugin>
+    </sensor>
+  </gazebo>
+  <gazebo reference="camera_link">
+    <material>Gazebo/Blue</material>
     <sensor type="depth" name="camera_link">
         <always_on>1</always_on>
@@ -116,211 +325,3 @@
     </sensor>
 </gazebo>
-  <joint name="camera_joint" type="continuous">
-    <axis xyz="0 0 1"/>
-    <parent link="body_link"/>
-    <child link="camera_link"/>
-    <origin rpy="0 0 0" xyz="0.2 0 -0.3"/>
-  </joint>
-  <link name="laser">
-    <visual>
-      <geometry>
-        <box size="0.0762 0.2794 0.0762"/>
-      </geometry>
-      <material name="blue">
-	<color rgba="0.1 0.1 1 1"/>
-      </material>
-    </visual>
-    <!--<collision>
-      <geometry>
-        <box size="0.0762 0.2794 0.0762"/>
-      </geometry>
-    </collision>-->
-   <inertial>
-      <mass value="0.25"/>
-      <inertia ixx="1.0" iyy="1.0" izz="1.0"
-               ixy="0" ixz="0" iyz="0"/>
-    </inertial>
-  </link>
-  <joint name="laser_joint" type="continuous">
-    <axis xyz="0 0 1"/>
-    <parent link="body_link"/>
-    <child link="laser"/>
-    <origin rpy="0 0 0" xyz="0.0 0 0.55"/>
-  </joint>
-  <link name="hitch_front_link">
-    <visual>
-      <geometry>
-        <cylinder length="0.1524" radius="0.01"/>
-      </geometry>
-      <material name="silver">
-	<color rgba="0.75 0.75 0.75 1"/>
-      </material>
-    </visual>
-    <collision>
-      <geometry>
-        <cylinder length="0.1524" radius="0.01"/>
-      </geometry>
-    </collision>
-    <inertial>
-      <mass value="0.1"/>
-      <inertia ixx="1.0" iyy="1.0" izz="1.0"
-               ixy="0" ixz="0" iyz="0"/>
-    </inertial>
-  </link>
-  <joint name="hitch_joint" type="fixed">
-    <axis xyz="0 0 1"/>
-    <parent link="base_link"/>
-    <child link="hitch_front_link"/>
-    <origin rpy="0 0 0" xyz="0.18 0 0.0762"/>
-  </joint>
-  <link name="wheel_front_left">
-    <visual>
-      <geometry>
-        <cylinder length="0.0508" radius="0.0762"/>
-      </geometry>
-      <material name="black">
-        <color rgba="0 0 0 1"/>
-      </material>
-    </visual>
-    <collision>
-      <geometry>
-        <cylinder length="0.0508" radius="0.0762"/>
-      </geometry>
-    </collision>
-    <inertial>
-      <mass value="0.1"/>
-      <inertia ixx="1.0" iyy="1.0" izz="1.0"
-               ixy="0" ixz="0" iyz="0"/>
-    </inertial>
-  </link>
-  <joint name="axis_front_left" type="continuous">
-    <axis xyz="0 0 1"/>
-    <parent link="base_link"/>
-    <child link="wheel_front_left"/>
-    <origin rpy="-1.5708 0 0" xyz="0.165862 0.18034 0"/>
-  </joint>
- <link name="wheel_front_right">
-    <visual>
-      <geometry>
-        <cylinder length="0.0508" radius="0.0762"/>
-      </geometry>
-      <material name="black"/>
-    </visual>
-    <collision>
-      <geometry>
-        <cylinder length="0.0508" radius="0.0762"/>
-      </geometry>
-    </collision>
-    <inertial>
-      <mass value="0.1"/>
-      <inertia ixx="1.0" iyy="1.0" izz="1.0"
-               ixy="0" ixz="0" iyz="0"/>
-    </inertial>
-  </link>
-  <joint name="axis_front_right" type="continuous">
-    <axis xyz="0 0 1"/>
-    <parent link="base_link"/>
-    <child link="wheel_front_right"/>
-    <origin rpy="-1.5708 0 0" xyz="0.165862 -0.18034 0"/>
-  </joint>
-  <link name="wheel_rear_right">
-    <visual>
-      <geometry>
-        <cylinder length="0.0508" radius="0.0762"/>
-      </geometry>
-      <material name="black"/>
-    </visual>
-    <collision>
-      <geometry>
-        <cylinder length="0.0508" radius="0.0762"/>
-      </geometry>
-    </collision>
-    <inertial>
-      <mass value="0.1"/>
-      <inertia ixx="1.0" iyy="1.0" izz="1.0"
-               ixy="0" ixz="0" iyz="0"/>
-    </inertial>
-  </link>
-  <joint name="axis_rear_right" type="continuous">
-    <axis xyz="0 0 1"/>
-    <parent link="base_link"/>
-    <child link="wheel_rear_right"/>
-    <origin rpy="-1.5708 0 0" xyz="-0.165862 -0.18034 0"/>
-  </joint>
-  <link name="wheel_rear_left">
-    <visual>
-      <geometry>
-        <cylinder length="0.0508" radius="0.0762"/>
-      </geometry>
-      <material name="black"/>
-    </visual>
-    <collision>
-      <geometry>
-        <cylinder length="0.0508" radius="0.0762"/>
-      </geometry>
-    </collision>
-    <inertial>
-      <mass value="0.1"/>
-      <inertia ixx="1.0" iyy="1.0" izz="1.0"
-               ixy="0" ixz="0" iyz="0"/>
-    </inertial>
-    <gazebo reference="wheel_rear_left">
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
Commit message: Fixed launch files

File: ros/urdf/efim.urdf.xacro (robot description, xacro)
@@ -74,5 +74,5 @@
     </inertial>
   </link>
-  <joint name="camera_joint" type="continuous">
+  <joint name="camera_joint" type="fixed">
     <axis xyz="0 0 0"/>
     <parent link="body_link"/>

Commit message: update

File: ros/urdf/efim.urdf.xacro (robot description, xacro)
@@ -83,5 +83,5 @@
     <visual>
       <geometry>
-        <box size="0.0762 0.2794 0.0762"/>
+        <box size="0.0762 0.0762 0.0762"/>
       </geometry>
       <material name="blue">
@@ -104,5 +104,5 @@
     <parent link="body_link"/>
     <child link="laser"/>
-    <origin rpy="0 0 0" xyz="0.0 0 0.55"/>
+    <origin rpy="0 0 0" xyz="0.0 0 0.75"/>
   </joint>
   <link name="hitch_front_link">
